File: pcbs/interposer/Interposer.sch (EAGLE design)
At the start: 21 parts

Commit message: Connected everything in schem except prototyping headers. Edited STMCubeMX project to reflect several new pin assignments.
Parts:
- added SJ1, SJ2: (no value), jumper:SJ
Connections:
- removed net BAT_VOLTAGE_SENSE: R1.1, R2.2
- removed net BNO_RST: JP10.6
- removed net ESTOP_ACTIVELOW: JP9.6
- removed net N$5: JP1.GPIO27, JP2.13
- removed net N$6: JP1.GPIO17, JP2.11
- new net BATT_SENSE: R1.1, R2.2, U$1.PA1
- new net BNO_RST_L: JP10.6, U$1.PE4
- new net ESTOP_L: JP9.6, U$1.PE2
- new net N$16: SJ1.2, U$1.PC2
- new net N$17: SJ2.1, U$1.PC1
- new net RPI_GPIO_IN: JP1.GPIO17, JP2.11, SJ2.2
- new net RPI_GPIO_OUT: JP1.GPIO27, JP2.13, SJ1.1
- net BNO_SCL: now also U$1.PB8
- net BNO_SDA: now also U$1.PB9
- net ESC1: now also U$1.PB4
- net ESC2: now also U$1.PC7
- net ESC3: now also U$1.PC8
- net ESC4: now also U$1.PC9
- net GPS_EN: now also U$1.PE5
- net GPS_FIX: now also U$1.PE6
- net GPS_RX: now also U$1.PB6
- net GPS_TX: now also U$1.PB7
- net RPI_RXD: now also U$1.PC10
- net RPI_TXD: now also U$1.PC11
- net SERVO_SIG: now also U$1.PA15
Other:
- moved on the sheet: JP10, JP11, JP12, JP13, JP2, JP3, JP4, JP5, JP6, JP7, JP8, JP9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

Commit message: Added a couple extra prototyping headers.
Parts:
- added JP14: t2ch4, pinhead:PINHD-1X3
- added JP15: t1ch1, pinhead:PINHD-1X3
- added JP16: t1ch2, pinhead:PINHD-1X3
- added JP17: t1ch3, pinhead:PINHD-1X3
- added JP18: t1ch4, pinhead:PINHD-1X3
- added JP19: POWproto, pinhead:PINHD-1X5
- added JP20: GNDproto, pinhead:PINHD-1X5
- JP7: value servo -> camServo
Connections:
- new net +V: JP19.4, JP19.5, JP8.2
- new net CAM_SERVO: JP7.1
- new net TIM1_CH1: JP15.1, U$1.PE9
- new net TIM1_CH2: JP16.1, U$1.PE11
- new net TIM1_CH3: JP17.1, U$1.PE13
- new net TIM1_CH4: JP18.1, U$1.PE14
- new net TIM2_CH4: JP14.1, U$1.PB11
- net +5V: now also JP14.2, JP15.2, JP16.2, JP17.2, JP18.2; no longer JP8.2
- net EGND: now also JP14.3, JP15.3, JP16.3, JP17.3, JP18.3, JP20.1, JP20.2, JP20.3, JP20.4, JP20.5
- net RPI_5V: now also JP19.1
- net SERVO_SIG: no longer JP7.1
- net STM5V: now also JP19.2, JP19.3
Other:
- moved on the sheet: JP7, JP8, JP9, R1, R2

Commit message: Edited the footprint with a script to connect the proto headers. Swapped sch/brd to use proto version of STM32. Fixed a bug with STM part pin numbering.
Parts:
- removed JP3, JP4: (no value), pinhead:PINHD-2X25
- U$1: value STM32F407DISCOVERY -> STM32F407DISCOVERYSTM32F407DISC-PROTO; device Interposer:STM32F407DISCOVERY -> Interposer:STM32F407DISCOVERYSTM32F407DISC-PROTO
Connections:
- net RPI_5V: now also JP19.2
- net STM5V: no longer JP19.2
Other:
- moved on the sheet: U$1
Changed lines of the file:
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@@
 <part name="JP1" library="AdafruitCobbler" deviceset="MICROBUILDER_RASBERRYPI_IDC" device=""/>
 <part name="JP2" library="pinhead" library_urn="urn:adsk.eagle:library:325" deviceset="PINHD-2X13" device="" package3d_urn="urn:adsk.eagle:package:22418/2"/>
-<part name="JP3" library="pinhead" library_urn="urn:adsk.eagle:library:325" deviceset="PINHD-2X25" device="" package3d_urn="urn:adsk.eagle:package:22454/2"/>
-<part name="JP4" library="pinhead" library_urn="urn:adsk.eagle:library:325" deviceset="PINHD-2X25" device="" package3d_urn="urn:adsk.eagle:package:22454/2"/>
 <part name="SUPPLY1" library="Power_Symbols" library_urn="urn:adsk.eagle:library:16502351" deviceset="EGND" device=""/>
 <part name="SUPPLY2" library="Power_Symbols" library_urn="urn:adsk.eagle:library:16502351" deviceset="EGND" device=""/>
 <part name="SUPPLY4" library="Power_Symbols" library_urn="urn:adsk.eagle:library:16502351" deviceset="+5V" device=""/>
-<part name="U$1" library="Interposer" deviceset="STM32F407DISCOVERY" device=""/>
+<part name="U$1" library="Interposer" deviceset="STM32F407DISCOVERY" device="STM32F407DISC-PROTO" value="STM32F407DISCOVERYSTM32F407DISC-PROTO"/>
 <part name="JP5" library="jumper" library_urn="urn:adsk.eagle:library:252" deviceset="JP1Q" device="" package3d_urn="urn:adsk.eagle:package:15455/1"/>
 <part name="JP6" library="jumper" library_urn="urn:adsk.eagle:library:252" deviceset="JP1Q" device="" package3d_urn="urn:adsk.eagle:package:15455/1"/>
@@
 <attribute name="VALUE" x="-133.35" y="7.62" size="1.778" layer="96"/>
 </instance>
-<instance part="JP3" gate="A" x="190.5" y="25.4" smashed="yes">
-<attribute name="NAME" x="184.15" y="59.055" size="1.778" layer="95"/>
-<attribute name="VALUE" x="184.15" y="-10.16" size="1.778" layer="96"/>
-</instance>
-<instance part="JP4" gate="A" x="231.14" y="25.4" smashed="yes">
-<attribute name="NAME" x="224.79" y="59.055" size="1.778" layer="95"/>
-<attribute name="VALUE" x="224.79" y="-10.16" size="1.778" layer="96"/>
-</instance>
 <instance part="SUPPLY1" gate="G$1" x="-66.04" y="55.88" smashed="yes">
 <attribute name="VALUE" x="-70.485" y="51.181" size="1.778" layer="96"/>
@@
 <segment>
 <pinref part="JP19" gate="A" pin="1"/>
-<wire x1="-121.92" y1="0" x2="-132.08" y2="0" width="0.1524" layer="91"/>
+<wire x1="-121.92" y1="0" x2="-129.54" y2="0" width="0.1524" layer="91"/>
 <label x="-132.08" y="0" size="1.778" layer="95" rot="R180" xref="yes"/>
+<pinref part="JP19" gate="A" pin="2"/>
+<wire x1="-129.54" y1="0" x2="-132.08" y2="0" width="0.1524" layer="91"/>
+<wire x1="-121.92" y1="-2.54" x2="-129.54" y2="-2.54" width="0.1524" layer="91"/>
+<wire x1="-129.54" y1="-2.54" x2="-129.54" y2="0" width="0.1524" layer="91"/>
+<junction x="-129.54" y="0"/>
 </segment>
 </net>
@@
 <segment>
 <pinref part="JP19" gate="A" pin="3"/>
-<wire x1="-121.92" y1="-5.08" x2="-129.54" y2="-5.08" width="0.1524" layer="91"/>
-<pinref part="JP19" gate="A" pin="2"/>
-<wire x1="-129.54" y1="-5.08" x2="-132.08" y2="-5.08" width="0.1524" layer="91"/>
-<wire x1="-121.92" y1="-2.54" x2="-129.54" y2="-2.54" width="0.1524" layer="91"/>
-<wire x1="-129.54" y1="-2.54" x2="-129.54" y2="-5.08" width="0.1524" layer="91"/>
-<junction x="-129.54" y="-5.08"/>
+<wire x1="-121.92" y1="-5.08" x2="-132.08" y2="-5.08" width="0.1524" layer="91"/>
 <label x="-132.08" y="-5.08" size="1.778" layer="95" rot="R180" xref="yes"/>
 </segment>

Commit message: Working through layout. Fixed a schematic bug and improved a few things.
Parts:
- JP19: value POWproto -> RP,RP,ST,VI,VI
- JP5: value (none) -> RPi5V
- renumbered R1 to R1_HIGH, R2 to R2_LOW
Connections:
- removed net +V: JP19.4, JP19.5, JP8.2
- removed net SERVO_SIG: U$1.PA15
- net +5V: now also JP19.4, JP19.5, JP8.2
- net CAM_SERVO: now also U$1.PA15
- net EGND: now also JP8.1

Commit message: Finished interposer board.
Parts:
- JP12: value GPS_5Vsrc_sel -> GPS_5Vsrc
- JP14, JP15, JP16, JP17, JP18, JP7: device pinhead:PINHD-1X3 -> Interposer:PINHD-1X3
- JP19, JP20: device pinhead:PINHD-1X5 -> Interposer:PINHD-1X5
- JP6: value (none) -> STM_PWR
Changed lines of the file:
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@@
 <part name="U$1" library="Interposer" deviceset="STM32F407DISCOVERY" device="STM32F407DISC-PROTO" value="STM32F407DISCOVERYSTM32F407DISC-PROTO"/>
 <part name="JP5" library="jumper" library_urn="urn:adsk.eagle:library:252" deviceset="JP1Q" device="" package3d_urn="urn:adsk.eagle:package:15455/1" value="RPi5V"/>
-<part name="JP6" library="jumper" library_urn="urn:adsk.eagle:library:252" deviceset="JP1Q" device="" package3d_urn="urn:adsk.eagle:package:15455/1"/>
+<part name="JP6" library="jumper" library_urn="urn:adsk.eagle:library:252" deviceset="JP1Q" device="" package3d_urn="urn:adsk.eagle:package:15455/1" value="STM_PWR"/>
 <part name="SUPPLY3" library="Power_Symbols" library_urn="urn:adsk.eagle:library:16502351" deviceset="+5V" device=""/>
 <part name="SUPPLY5" library="Power_Symbols" library_urn="urn:adsk.eagle:library:16502351" deviceset="EGND" device=""/>
 <part name="SUPPLY6" library="Power_Symbols" library_urn="urn:adsk.eagle:library:16502351" deviceset="+V" device="" value="+3V"/>
-<part name="JP7" library="pinhead" library_urn="urn:adsk.eagle:library:325" deviceset="PINHD-1X3" device="" package3d_urn="urn:adsk.eagle:package:22458/2" value="camServo"/>
+<part name="JP7" library="Interposer" deviceset="PINHD-1X3" device="" package3d_urn="urn:adsk.eagle:package:22458/2" value="camServo"/>
 <part name="JP8" library="pinhead" library_urn="urn:adsk.eagle:library:325" deviceset="PINHD-1X3" device="" package3d_urn="urn:adsk.eagle:package:22458/2" value="power"/>
 <part name="JP9" library="pinhead" library_urn="urn:adsk.eagle:library:325" deviceset="PINHD-1X8" device="" package3d_urn="urn:adsk.eagle:package:22409/2" value="EStopBrd_cable"/>
@@
 <part name="U$32" library="microbuilder" deviceset="MOUNTINGHOLE" device="2.5_THICK"/>
 <part name="SUPPLY10" library="Power_Symbols" library_urn="urn:adsk.eagle:library:16502351" deviceset="EGND" device=""/>
-<part name="JP12" library="pinhead" library_urn="urn:adsk.eagle:library:325" deviceset="PINHD-1X3" device="" package3d_urn="urn:adsk.eagle:package:22458/2" value="GPS_5Vsrc_sel"/>
+<part name="JP12" library="pinhead" library_urn="urn:adsk.eagle:library:325" deviceset="PINHD-1X3" device="" package3d_urn="urn:adsk.eagle:package:22458/2" value="GPS_5Vsrc"/>
 <part name="SUPPLY11" library="Power_Symbols" library_urn="urn:adsk.eagle:library:16502351" deviceset="+5V" device=""/>
 <part name="JP13" library="pinhead" library_urn="urn:adsk.eagle:library:325" deviceset="PINHD-1X9" device="" package3d_urn="urn:adsk.eagle:package:22483/2" value="GPS_module"/>
@@
 <part name="SUPPLY13" library="Power_Symbols" library_urn="urn:adsk.eagle:library:16502351" deviceset="EGND" device=""/>
 <part name="SUPPLY14" library="Power_Symbols" library_urn="urn:adsk.eagle:library:16502351" deviceset="+5V" device=""/>
-<part name="JP14" library="pinhead" library_urn="urn:adsk.eagle:library:325" deviceset="PINHD-1X3" device="" package3d_urn="urn:adsk.eagle:package:22458/2" value="t2ch4"/>
-<part name="JP15" library="pinhead" library_urn="urn:adsk.eagle:library:325" deviceset="PINHD-1X3" device="" package3d_urn="urn:adsk.eagle:package:22458/2" value="t1ch1"/>
-<part name="JP16" library="pinhead" library_urn="urn:adsk.eagle:library:325" deviceset="PINHD-1X3" device="" package3d_urn="urn:adsk.eagle:package:22458/2" value="t1ch2"/>
-<part name="JP17" library="pinhead" library_urn="urn:adsk.eagle:library:325" deviceset="PINHD-1X3" device="" package3d_urn="urn:adsk.eagle:package:22458/2" value="t1ch3"/>
-<part name="JP18" library="pinhead" library_urn="urn:adsk.eagle:library:325" deviceset="PINHD-1X3" device="" package3d_urn="urn:adsk.eagle:package:22458/2" value="t1ch4"/>
-<part name="JP20" library="pinhead" library_urn="urn:adsk.eagle:library:325" deviceset="PINHD-1X5" device="" package3d_urn="urn:adsk.eagle:package:22469/2" value="GNDproto"/>
-<part name="JP19" library="pinhead" library_urn="urn:adsk.eagle:library:325" deviceset="PINHD-1X5" device="" package3d_urn="urn:adsk.eagle:package:22469/2" value="RP,RP,ST,VI,VI"/>
+<part name="JP14" library="Interposer" deviceset="PINHD-1X3" device="" package3d_urn="urn:adsk.eagle:package:22458/2" value="t2ch4"/>
+<part name="JP15" library="Interposer" deviceset="PINHD-1X3" device="" package3d_urn="urn:adsk.eagle:package:22458/2" value="t1ch1"/>
+<part name="JP16" library="Interposer" deviceset="PINHD-1X3" device="" package3d_urn="urn:adsk.eagle:package:22458/2" value="t1ch2"/>
+<part name="JP17" library="Interposer" deviceset="PINHD-1X3" device="" package3d_urn="urn:adsk.eagle:package:22458/2" value="t1ch3"/>
+<part name="JP18" library="Interposer" deviceset="PINHD-1X3" device="" package3d_urn="urn:adsk.eagle:package:22458/2" value="t1ch4"/>
+<part name="JP20" library="Interposer" deviceset="PINHD-1X5" device="" package3d_urn="urn:adsk.eagle:package:22469/2" value="GNDproto"/>
+<part name="JP19" library="Interposer" deviceset="PINHD-1X5" device="" package3d_urn="urn:adsk.eagle:package:22469/2" value="RP,RP,ST,VI,VI"/>
 </parts>
 <sheets>

Commit message: Increased e-stop <-> interposer ribbon cable drill size to make soldering the ribbon cable easier in future versions.
Parts:
- JP9: device pinhead:PINHD-1X8 -> HighCurrentTransistorAndDriver:PINHD-1X8_RIBBONCABLE
Changed lines of the file:
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@@
 <part name="JP7" library="Interposer" deviceset="PINHD-1X3" device="" package3d_urn="urn:adsk.eagle:package:22458/2" value="camServo"/>
 <part name="JP8" library="pinhead" library_urn="urn:adsk.eagle:library:325" deviceset="PINHD-1X3" device="" package3d_urn="urn:adsk.eagle:package:22458/2" value="power"/>
-<part name="JP9" library="pinhead" library_urn="urn:adsk.eagle:library:325" deviceset="PINHD-1X8" device="" package3d_urn="urn:adsk.eagle:package:22409/2" value="EStopBrd_cable"/>
+<part name="JP9" library="HighCurrentTransistorAndDriver" deviceset="PINHD-1X8_RIBBONCABLE" device="" package3d_urn="urn:adsk.eagle:package:22409/2" value="EStopBrd_cable"/>
 <part name="R1_HIGH" library="adafruit" library_urn="urn:adsk.eagle:library:420" deviceset="R-US_" device="0204/7" package3d_urn="urn:adsk.eagle:package:6240596/1"/>
 <part name="R2_LOW" library="adafruit" library_urn="urn:adsk.eagle:library:420" deviceset="R-US_" device="0204/7" package3d_urn="urn:adsk.eagle:package:6240596/1"/>
